File: Hardware/Vmeasure/Vmeasure.kicad_pcb (KiCad board)
At the start: 2 copper layers, 110 x 65 mm, 41 parts, among them J1 Conn_Coaxial, J2 Conn_Coaxial, J3 Conn_Coaxial, J4 Conn_Coaxial, U3 ADS1248IPWR, U4 REF5040AD, U7 SC0915

Commit message: little update
Parts:
- added D10: LED, LED_SMD:LED_PLCC-2, F.Cu at (190.0, 57.2)
- added D11: LED, LED_SMD:LED_PLCC-2, F.Cu at (205.2, 34.4)
- added D12: LED, LED_SMD:LED_PLCC-2, F.Cu at (211.4, 34.4)
- added D9: LED, LED_SMD:LED_PLCC-2, F.Cu at (190.0, 52.5)
- added Debug1: Conn_01x04, Connector_JST:JST_XH_B4B-XH-A_1x04_P2.50mm_Vertical, F.Cu at (157.5, 30.0)
- added I2C1: Conn_01x04, Connector_JST:JST_XH_B4B-XH-A_1x04_P2.50mm_Vertical, F.Cu at (100.0, 130.0)
- added I2C2: Conn_01x04, Connector_JST:JST_XH_B4B-XH-A_1x04_P2.50mm_Vertical, F.Cu at (180.8, 45.7)
- added PWRin1: Conn_01x02, Connector_JST:JST_XH_B2B-XH-A_1x02_P2.50mm_Vertical, F.Cu at (262.5, 40.0)
- added R27: 0R, Resistor_SMD:R_0805_2012Metric_Pad1.20x1.40mm_HandSolder, F.Cu at (142.3, 117.2)
- added R28: 0R, Resistor_SMD:R_0805_2012Metric_Pad1.20x1.40mm_HandSolder, F.Cu at (142.3, 112.6)
- added R29: 0R, Resistor_SMD:R_0805_2012Metric_Pad1.20x1.40mm_HandSolder, F.Cu at (142.3, 108.1)
- added R30: 0R, Resistor_SMD:R_0805_2012Metric_Pad1.20x1.40mm_HandSolder, F.Cu at (137.5, 35.0)
- added R31: 0R, Resistor_SMD:R_0805_2012Metric_Pad1.20x1.40mm_HandSolder, F.Cu at (147.5, 35.0)
- added R32: 0R, Resistor_SMD:R_0805_2012Metric_Pad1.20x1.40mm_HandSolder, F.Cu at (167.2, 117.2)
- added R33: 0R, Resistor_SMD:R_0805_2012Metric_Pad1.20x1.40mm_HandSolder, F.Cu at (192.3, 117.2)
- added R34: 0R, Resistor_SMD:R_0805_2012Metric_Pad1.20x1.40mm_HandSolder, F.Cu at (167.2, 112.6)
- added R35: 0R, Resistor_SMD:R_0805_2012Metric_Pad1.20x1.40mm_HandSolder, F.Cu at (192.3, 112.6)
- added R36: 0R, Resistor_SMD:R_0805_2012Metric_Pad1.20x1.40mm_HandSolder, F.Cu at (217.2, 117.2)
- added R37: 0R, Resistor_SMD:R_0805_2012Metric_Pad1.20x1.40mm_HandSolder, F.Cu at (167.2, 108.1)
- added R38: 0R, Resistor_SMD:R_0805_2012Metric_Pad1.20x1.40mm_HandSolder, F.Cu at (192.3, 108.1)
- added R39: 0R, Resistor_SMD:R_0805_2012Metric_Pad1.20x1.40mm_HandSolder, F.Cu at (217.2, 112.6)
- added R40: 0R, Resistor_SMD:R_0805_2012Metric_Pad1.20x1.40mm_HandSolder, F.Cu at (217.2, 108.1)
- added R41: 0R, Resistor_SMD:R_0805_2012Metric_Pad1.20x1.40mm_HandSolder, F.Cu at (204.4, 38.2)
- added R42: 0R, Resistor_SMD:R_0805_2012Metric_Pad1.20x1.40mm_HandSolder, F.Cu at (209.1, 38.2)
- added R43: 47R, Resistor_SMD:R_0805_2012Metric_Pad1.20x1.40mm_HandSolder, F.Cu at (262.4, 77.2)
- added R44: 47R, Resistor_SMD:R_0805_2012Metric_Pad1.20x1.40mm_HandSolder, F.Cu at (259.0, 71.3)
- added R45: 47R, Resistor_SMD:R_0805_2012Metric_Pad1.20x1.40mm_HandSolder, F.Cu at (265.2, 68.0)
- added R46: 47R, Resistor_SMD:R_0805_2012Metric_Pad1.20x1.40mm_HandSolder, F.Cu at (251.5, 81.4)
- added R47: 0R, Resistor_SMD:R_0805_2012Metric_Pad1.20x1.40mm_HandSolder, F.Cu at (252.9, 78.0)
- added R48: 0R, Resistor_SMD:R_0805_2012Metric_Pad1.20x1.40mm_HandSolder, F.Cu at (259.0, 74.3)
- added R49: 0R, Resistor_SMD:R_0805_2012Metric_Pad1.20x1.40mm_HandSolder, F.Cu at (263.8, 71.3)
- added R50: 0R, Resistor_SMD:R_0805_2012Metric_Pad1.20x1.40mm_HandSolder, F.Cu at (257.6, 78.0)
- added R51: 47R, Resistor_SMD:R_0805_2012Metric_Pad1.20x1.40mm_HandSolder, F.Cu at (269.9, 68.0)
- added R52: 47R, Resistor_SMD:R_0805_2012Metric_Pad1.20x1.40mm_HandSolder, F.Cu at (256.2, 81.0)
- added R53: 0R, Resistor_SMD:R_0805_2012Metric_Pad1.20x1.40mm_HandSolder, F.Cu at (263.8, 74.3)
- added R54: 0R, Resistor_SMD:R_0805_2012Metric_Pad1.20x1.40mm_HandSolder, F.Cu at (268.5, 70.9)
- added R55: 0R, Resistor_SMD:R_0805_2012Metric_Pad1.20x1.40mm_HandSolder, F.Cu at (246.7, 81.4)
- added R56: 0R, Resistor_SMD:R_0805_2012Metric_Pad1.20x1.40mm_HandSolder, F.Cu at (262.4, 80.2)
- added R57: 47R, Resistor_SMD:R_0805_2012Metric_Pad1.20x1.40mm_HandSolder, F.Cu at (268.5, 73.9)
- added R58: 470k, Resistor_SMD:R_0805_2012Metric_Pad1.20x1.40mm_HandSolder, F.Cu at (267.1, 77.2)
- added R59: 47R, Resistor_SMD:R_0805_2012Metric_Pad1.20x1.40mm_HandSolder, F.Cu at (267.1, 80.2)
- added TP1: TestPoint_2Pole, TestPoint:TestPoint_2Pads_Pitch2.54mm_Drill0.8mm, F.Cu at (246.2, 71.5)
- added TP2: TestPoint_2Pole, TestPoint:TestPoint_2Pads_Pitch2.54mm_Drill0.8mm, F.Cu at (252.3, 68.2)
- added TP3: TestPoint_2Pole, TestPoint:TestPoint_2Pads_Pitch2.54mm_Drill0.8mm, F.Cu at (246.2, 74.9)
- added TP4: TestPoint_2Pole, TestPoint:TestPoint_2Pads_Pitch2.54mm_Drill0.8mm, F.Cu at (252.3, 71.5)
- added TP5: TestPoint_2Pole, TestPoint:TestPoint_2Pads_Pitch2.54mm_Drill0.8mm, F.Cu at (258.5, 68.2)
- added TP6: TestPoint_2Pole, TestPoint:TestPoint_2Pads_Pitch2.54mm_Drill0.8mm, F.Cu at (246.2, 78.2)
- added TP7: TestPoint_2Pole, TestPoint:TestPoint_2Pads_Pitch2.54mm_Drill0.8mm, F.Cu at (252.3, 74.9)
- added TP8: TestPoint_2Pole, TestPoint:TestPoint_2Pads_Pitch2.54mm_Drill0.8mm, F.Cu at (254.3, 115.1)
- added U1: OPA2333xxDGK, Package_SO:VSSOP-8_3.0x3.0mm_P0.65mm, F.Cu at (151.6, 100.6)
- added U2: OPA2333xxDGK, Package_SO:VSSOP-8_3.0x3.0mm_P0.65mm, F.Cu at (204.0, 101.6)
- added U5: OPA2333xxDGK, Package_SO:VSSOP-8_3.0x3.0mm_P0.65mm, F.Cu at (231.0, 24.9)
- added U6: OPA2333xxDGK, Package_SO:VSSOP-8_3.0x3.0mm_P0.65mm, F.Cu at (231.0, 29.4)
- moved H7 120.5 mm to (125.0, 130.0)
- moved R13 116.8 mm to (142.3, 121.8), turned to 180 degrees
- moved R19 105.7 mm to (137.5, 105.8), turned to 270 degrees
- moved R4 105.0 mm to (137.5, 119.5), turned to 270 degrees
- moved H8 88.4 mm to (125.0, 75.0)
- moved U3 83.9 mm to (265.8, 112.2)
- moved R10 79.1 mm to (187.5, 114.9), turned to 270 degrees
- moved R8 75.6 mm to (137.5, 114.9), turned to 270 degrees
- moved R12 71.4 mm to (137.5, 110.4), turned to 270 degrees
- moved R6 71.0 mm to (187.5, 119.5), turned to 270 degrees
- moved R15 65.1 mm to (167.2, 121.8), turned to 180 degrees
- moved J1 64.3 mm to (137.5, 131.8)
- moved J2 64.3 mm to (162.5, 131.8)
- moved J4 64.3 mm to (212.5, 131.8)
- moved J3 64.3 mm to (187.5, 131.8)
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Connections:
- R13 pad 1: (no net) -> Net-(D5-Pad1)
- R15 pad 1: (no net) -> Net-(D6-Pad1)
- R17 pad 1: (no net) -> Net-(D7-Pad1)
- R23 pad 1: (no net) -> Net-(D8-Pad1)
- U3 pad 10: (no net) -> VREFCOM
- U3 pad 11: (no net) -> Net-(R53-Pad1)
- U3 pad 12: (no net) -> Net-(R47-Pad1)
- U3 pad 13: (no net) -> Net-(R55-Pad1)
- U3 pad 14: (no net) -> Net-(R49-Pad1)
- U3 pad 15: (no net) -> Net-(R56-Pad1)
- U3 pad 16: (no net) -> Net-(R50-Pad1)
- U3 pad 17: (no net) -> Net-(R54-Pad1)
- U3 pad 18: (no net) -> Net-(R48-Pad1)
- U3 pad 19: (no net) -> IEXC2
- U3 pad 2: (no net) -> GNDD
- U3 pad 20: (no net) -> IEXC1
- U3 pad 21: (no net) -> GNDA
- U3 pad 23: (no net) -> Net-(R46-Pad1)
- U3 pad 24: (no net) -> Net-(R51-Pad1)
- U3 pad 25: (no net) -> Net-(R57-Pad2)
- U3 pad 26: (no net) -> Net-(R59-Pad2)
- U3 pad 27: (no net) -> Net-(R43-Pad1)
- U3 pad 28: (no net) -> Net-(R52-Pad1)
- U3 pad 3: (no net) -> Net-(R44-Pad1)
- U3 pad 4: (no net) -> Net-(R45-Pad1)
- U3 pad 5: (no net) -> REFP0
- U3 pad 6: (no net) -> REFN0
- U3 pad 7: (no net) -> REFP1
- U3 pad 8: (no net) -> REFN1
- U3 pad 9: (no net) -> VREFOUT
- U7 pad 13: Net-(U7-Pad13) -> GNDD
- U7 pad 18: Net-(U7-Pad13) -> GNDD
- U7 pad 23: Net-(U7-Pad13) -> GNDD
- U7 pad 28: Net-(U7-Pad13) -> GNDD
- U7 pad 3: Net-(U7-Pad13) -> GNDD
- U7 pad 38: Net-(U7-Pad13) -> GNDD
- U7 pad 8: Net-(U7-Pad13) -> GNDD
- U7 pad D2: Net-(U7-Pad13) -> GNDD
Routing:
- net Net-(D8-Pad1): track 0.00 -> 13.7 mm
- net Net-(D7-Pad1): track 0.00 -> 13.7 mm
- net Net-(D6-Pad1): track 0.00 -> 13.7 mm
- net Net-(D5-Pad1): track 0.00 -> 13.7 mm
- net Net-(R10-Pad2): track 0.00 -> 7.51 mm
- net Net-(D2-Pad1): track 0.00 -> 7.50 mm
- net Net-(D4-Pad1): track 0.00 -> 7.48 mm
- net Net-(D1-Pad1): track 0.00 -> 7.47 mm
- net Net-(D3-Pad1): track 0.00 -> 7.46 mm
- net Net-(R17-Pad2): track 0.00 -> 6.70 mm
- net Net-(R11-Pad2): track 0.00 -> 6.66 mm
- net Net-(R16-Pad1): track 0.00 -> 6.62 mm
- net Net-(R32-Pad2): track 0.00 -> 6.61 mm
- net Net-(R22-Pad1): track 0.00 -> 6.59 mm
- net Net-(R15-Pad2): track 0.00 -> 6.50 mm
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Other:
- board size 110 x 65 mm -> 150 x 65 mm
