File: Hardware/Vmeasure/Vmeasure.sch (KiCad schematic (older format))
At the start: 56 parts

Commit message: PCB outline and connector placement
Parts:
- added D? (x2): LED, LED_SMD:LED_PLCC-2, symbol Device:LED
- added H1, H2, H3, H4, H5, H6, H7, H8: MountingHole, MountingHole:MountingHole_3.2mm_M3_DIN965_Pad_TopBottom, symbol Mechanical:MountingHole
- added R? (x2): 0R, Resistor_SMD:R_0805_2012Metric_Pad1.20x1.40mm_HandSolder, symbol Device:R_Small
- Debug1: renamed from Debug; footprint (none) -> Connector_JST:JST_XH_B4B-XH-A_1x04_P2.50mm_Vertical
- I2C1: renamed from I2C; footprint (none) -> Connector_JST:JST_XH_B4B-XH-A_1x04_P2.50mm_Vertical
- I2C2: renamed from I2C?; footprint (none) -> Connector_JST:JST_XH_B4B-XH-A_1x04_P2.50mm_Vertical
- PWRin1: renamed from PWRin; footprint (none) -> Connector_JST:JST_XH_B2B-XH-A_1x02_P2.50mm_Vertical
- gave numbers to parts that had none: 45
Other:
- note added: "mech range switch?\n"

Commit message: little update
Parts:
- added D11, D12: LED, LED_SMD:LED_PLCC-2, symbol Device:LED
- added R27, R28, R29, R32, R33, R34, R35, R36, R37, R38, R39, R40, R41, R42, R47, R48, R49, R50, R53, R54, R55, R56: 0R, Resistor_SMD:R_0805_2012Metric_Pad1.20x1.40mm_HandSolder, symbol Device:R_Small
- added R43, R44, R45, R46, R51, R52, R57, R59: 47R, Resistor_SMD:R_0805_2012Metric_Pad1.20x1.40mm_HandSolder, symbol Device:R_Small
- added R58: 470k, Resistor_SMD:R_0805_2012Metric_Pad1.20x1.40mm_HandSolder, symbol Device:R_Small
- added TP1, TP2, TP3, TP4, TP5, TP6, TP7, TP8: TestPoint_2Pole, TestPoint:TestPoint_2Pads_Pitch2.54mm_Drill0.8mm, symbol Connector:TestPoint_2Pole
- U1, U2, U5, U6: footprint (none) -> Package_SO:VSSOP-8_3.0x3.0mm_P0.65mm
- gave numbers to parts that had none: 4
Connections:
- net AIN0: now also R53.2
- net AIN2: now also R54.2
- net AIN4: now also R55.2; no longer U2.1
- net VDD: now reaches U3.1 (DVDD)
- net VREFCOM: now reaches U3.10 (VREFCOM)
- net VREFCOM: now also TP5.2
- net at U3.11 (AIN0/IEXC): now also R53.1
- net at U3.12 (AIN1/IEXC): now also R47.1
- net at U3.13 (AIN4/IEXC/GPIO4): now also R55.1
- net at U3.14 (AIN5/IEXC/GPIO5): now also R49.1
- net at U3.15 (AIN6/IEXC/GPIO6): now also R56.1
- net at U3.16 (AIN7/IEXC/GPIO7): now also R50.1
- net at U3.17 (AIN2/IEXC/GPIO2): now also R54.1
- net at U3.18 (AIN3/IEXC/GPIO3): now also R48.1
- net IEXC2: now reaches U3.19 (IEXC2)
- net IEXC2: now also TP3.2
- net GNDD: now reaches U3.2 (DGND)
- net GNDD: now also D10.1 (K), D9.1 (K), U7.13 (GND), U7.18 (GND), U7.23 (GND), U7.28 (GND), U7.3 (GND), U7.38 (GND), U7.8 (GND), U7.D2 (GND), D11.1 (K), D12.1 (K)
- net IEXC1: now reaches U3.20 (IEXC1)
- net IEXC1: now also TP2.2
- net GNDA: now reaches U3.21 (AVSS)
- net GNDA: now also TP1.1, TP2.1, TP3.1, TP4.1, TP5.1, TP6.1, TP7.1, TP8.1
- net VDDA: now reaches U3.22 (AVDD)
- net at U3.23 (START): now also R46.1
- net at U3.24 (~CS): now also R51.1
- net at U3.25 (~DRDY): now also R57.2
- net at U3.26 (DOUT/~DRDY): now also R59.2
- net at U3.27 (DIN): now also R43.1
- net at U3.28 (SCLK): now also R52.1
- net at U3.3 (CLK): now also R44.1
- net at U3.4 (~RESET): now also R45.1
- net REFP0: now reaches U3.5 (REFP0/GPIO0)
- net REFP0: now also TP1.2
- net REFN0: now reaches U3.6 (REFN0/GPIO1)
- net REFN0: now also TP4.2
- net REFP1: now reaches U3.7 (REFP1)
- net REFP1: now also TP7.2
- net REFN1: now reaches U3.8 (REFN1)
- net REFN1: now also TP8.2
- net VREFOUT: now reaches U3.9 (VREFOUT)
- net VREFOUT: now also TP6.2
- net AIN1: now reaches U1.1, U1.2 (-)
- net AIN1: now also R47.2
- net at D5.1 (A1), R13.1, U1.3 (+): now also R27.1, R28.1, R29.1
- net at U1.5 (+): now also D6.1 (A1), R15.1, R32.1, R34.1, R37.1
- net AIN3: now reaches U1.6 (-)
- net AIN3: now also U1.7, R48.2
- net at R4.1, R8.2: now also R27.2
- net at R12.2, R8.1: now also R28.2
- net at R12.1, R19.2: now also R29.2
- net AIN5: now reaches U2.2 (-)
- net AIN5: now also U2.1, R49.2
- net at D7.1 (A1), R17.1, U2.3 (+): now also R33.1, R35.1, R38.1
- net at D8.1 (A1), R23.1, U2.5 (+): now also R36.1, R39.1, R40.1
- net AIN7: now reaches U2.6 (-)
- net AIN7: now also U2.7, R50.2
- net at R5.1, R9.2: now also R32.2
- net at R14.2, R9.1: now also R34.2
- net at R14.1, R20.2: now also R37.2
- net at R10.2, R6.1: now also R33.2
- net at R10.1, R16.2: now also R35.2
- net at R16.1, R21.2: now also R38.2
- net at R11.1, R18.2: now also R36.2
- net at R18.1, R22.2: now also R39.2
- net at R22.1, R24.2: now also R40.2
- net at D9.2 (A): now also R30.2
- net at D10.2 (A): now also R31.2
- net Ain6 renamed AIN6
- net AIN6: now also R56.2
- new net: D11.2 (A), R41.2
- new net: D12.2 (A), R42.2
- new net CLK: R44.2
- new net CS: R51.2
- new net DIN: R43.2
- new net DOUT: R59.1
- new net DRDY: R57.1
- new net RST: R45.2
- new net SCLK: R52.2
- new net START: R46.2
Other:
- note removed: "mech range switch?\n"
